File: RTD/16_channel_RTD/16_channel_RTD.kicad_sch (KiCad schematic)
At the start: 0 parts

Commit message: ERC free
Other:
- sheet Analog_Front_End ports: added none; removed EN
- sheet MCU ports: added HOLD, MISO, MOSI, NSS, SCK; removed EN
- sheet Non_Volatile_Memory ports: added HOLD, MISO, MOSI, NSS, SCK; removed none
